File: usb-c-to-liion-charger.kicad_pcb (KiCad board)
At the start: 2 copper layers, 98 x 39.5 mm, 73 parts, among them J1 USB_C_Receptacle_USB2.0, J2 BatteryConnection, Q1 RSJ250P10, Q2 RSJ250P10, Q3 BSC016N06NS, Q4 BSC016N06NS, SW1 SW_DPDT_x2, SW2 SW_SPDT, U1 IP2721, U2 LTC4000-QFN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

Commit message: Fix wrong battery polarity Enable voltage monitoring at 15V Add caps to OFB and BFB Use another diodes Replace 1206 shunt with 0805 Replace main mosfet with bigger one Improve traces/ground planes
Parts:
- added C23: 100nF, Capacitor_SMD:C_0603_1608Metric, B.Cu at (123.0, 94.9)
- added C24: 10nF, Capacitor_SMD:C_0603_1608Metric, F.Cu at (131.0, 101.2)
- added C25: 10nF, Capacitor_SMD:C_0603_1608Metric, F.Cu at (122.4, 107.7)
- added C26: 1nF, Capacitor_SMD:C_0603_1608Metric, F.Cu at (138.1, 89.7)
- added C27: 10nF, Capacitor_SMD:C_0603_1608Metric, F.Cu at (139.0, 87.4)
- added C28: 1uF 25V, Capacitor_SMD:C_0805_2012Metric, F.Cu at (153.6, 88.5)
- added C29: 100nF 25V, Capacitor_SMD:C_0805_2012Metric, F.Cu at (155.7, 88.5)
- added JP1: SolderJumper_2_Open, extraFootprints:SolderJumper-Open_0603, B.Cu at (141.2, 92.9)
- added JP2: SolderJumper_2_Open, extraFootprints:SolderJumper-Open_0603, B.Cu at (143.1, 89.9)
- added R29: 150k, Resistor_SMD:R_0603_1608Metric, B.Cu at (123.0, 97.9)
- added R30: 13k, Resistor_SMD:R_0603_1608Metric, B.Cu at (122.9, 96.4)
- added R31: 10k, Resistor_SMD:R_0603_1608Metric, F.Cu at (139.8, 89.7)
- added R32: 0R, Resistor_SMD:R_0603_1608Metric, B.Cu at (154.7, 94.5)
- added R33: 0R, Resistor_SMD:R_0603_1608Metric, B.Cu at (155.6, 89.5)
- C12: moved to B.Cu
- C18: value 100n -> 470nF 25V
- C3: value 47nF -> 100nF
- D4, D5: value CFSH05-20L -> MBR0580-TP; footprint extraFootprints:SOD882D -> Diode_SMD:D_SOD-123
- L1: footprint Inductor_SMD:L_Coilcraft_XAL60xx_6.36x6.56mm -> Inductor_SMD:L_Coilcraft_XAL6060-XXX
- Q3: value BSC016N06NS -> BSC047N08NS3 G
- Q4: value BSC016N06NS -> AOD66920; footprint Package_TO_SOT_SMD:TDSON-8-1 -> Package_TO_SOT_SMD:TO-252-3_TabPin2
- R13, R14, R26: footprint extraFootprints:R_1206_3216Metric_4Kelvin -> extraFootprints:R_0805_2012Metric_4Kelvin
- R25: moved to F.Cu
- R7: value 22k -> 15k
- moved C12 10.6 mm to (146.0, 88.5), turned to 180 degrees
- moved L1 8.04 mm to (163.3, 85.5), turned to 0 degrees
- moved C22 5.06 mm to (148.0, 97.2), turned to -90 degrees
- moved J2 5.00 mm to (191.3, 104.8), turned to 90 degrees
- moved D5 4.46 mm to (151.9, 93.1)
- moved C18 4.40 mm to (153.9, 92.1), turned to 90 degrees
- moved U3 4.25 mm to (147.1, 92.5)
- moved C17 3.65 mm to (143.0, 92.3)
- moved C20 3.59 mm to (151.6, 88.5)
- moved C19 3.51 mm to (149.6, 88.5)
- moved R25 3.27 mm to (144.2, 89.4)
- moved C21 2.73 mm to (146.1, 97.3), turned to -90 degrees
- moved Q3 2.61 mm to (163.2, 100.5)
- moved Q4 2.39 mm to (163.5, 92.9)
- moved C13 2.22 mm to (143.2, 101.2)
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Connections:
- C17 pad 1: /Boost-Converter/SS -> Net-(U3-SS)
- C2 pad 1: Net-(U2-CSP) -> /Charge-IC/CSP
- C5 pad 1: /Charge-IC/VIN -> Net-(U2-IN)
- C6 pad 1: /Charge-IC/VIN -> Net-(U2-IN)
- F2 pad 2: Net-(J2-Pin_1) -> Net-(J2-Pin_2)
- J2 pad 1: Net-(J2-Pin_1) -> GND
- J2 pad 2: GND -> Net-(J2-Pin_2)
- Q1 pad 3: /Charge-IC/CSP -> Net-(Q1-S)
- Q4 pad 1: GND -> Net-(Q4-G)
- Q4 pad 2: GND -> Net-(Q4-D)
- R13 pad 2: /Charge-IC/VIN -> Net-(U2-IN)
- R14 pad 1: /Charge-IC/CSP -> Net-(Q1-S)
- R14 pad 2: Net-(U2-CSP) -> /Charge-IC/CSP
- R25 pad 2: Net-(U3-RUN) -> /Boost-Converter/RUN
- R8 pad 2: /Charge-IC/CSP -> Net-(Q1-S)
- U2 pad 1: /Charge-IC/BIAS -> Net-(U2-VM)
- U2 pad 2: /Boost-Converter/SS -> /Boost-Converter/RUN
- U2 pad 20: Net-(U2-CSP) -> /Charge-IC/CSP
- U2 pad 27: /Charge-IC/VIN -> Net-(U2-IN)
- U3 pad 11: Net-(U3-RUN) -> /Boost-Converter/RUN
- U3 pad 12: /Boost-Converter/SS -> Net-(U3-SS)
- U3 pad 17: /Boost-Converter/INTV_{CC} -> Net-(JP2-B)
- U3 pad 19: Net-(Q3-G) -> Net-(U3-TG)
- U3 pad 21: Net-(Q4-G) -> Net-(U3-BG)
- U3 pad 9: /Boost-Converter/INTV_{CC} -> Net-(JP1-B)
Routing:
- net Net-(U2-CSP): track 61.0 -> 0.00 mm
- net GND: track 14.4 -> 60.5 mm, vias 116 -> 238
- net /Boost-Converter/SS: track 30.5 -> 0.00 mm, vias 3 -> 0
- net /Boost-Converter/RUN: track 0.00 -> 26.9 mm, vias 0 -> 3
- net /Charge-IC/CSP: track 54.6 -> 75.7 mm, vias 4 -> 2
- net Net-(J2-Pin_2): track 0.00 -> 11.8 mm
- net Net-(J2-Pin_1): track 10.7 -> 0.00 mm
- net /Boost-Converter/INTV_{CC}: track 93.5 -> 84.3 mm, vias 3 -> 1
- net Net-(Q4-G): track 11.2 -> 2.76 mm, vias 3 -> 1
- net /Charge-IC/BIAS: track 26.7 -> 18.4 mm, vias 2 -> 0
- net Net-(U2-VM): track 0.00 -> 8.21 mm, vias 0 -> 1
- net Net-(U3-BG): track 0.00 -> 8.11 mm
- net Net-(U2-IN): track 0.00 -> 7.78 mm
- net Net-(Q3-G): track 14.9 -> 7.13 mm
- net Net-(U3-TG): track 0.00 -> 6.70 mm, vias 0 -> 2
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- added copper zone on F.Cu, net Net-(Q1-S)
- removed copper zone on F.Cu, net /Charge-IC/CSP
Other:
- board size 98 x 39.5 mm -> 98 x 42 mm
- board text added: "USB-C PD to 10S/12S Li-Ion charger v1.1 2023-03 by MG"
- board text removed: "USB-C PD to 10S/12S Li-Ion charger v1.0 2022-05 by MG"
