File: usb-c-to-liion-charger.kicad_sch (KiCad schematic)
At the start: 15 parts, among them J1 USB_C_Receptacle_USB2.0, J2 BatteryConnection, U1 IP2721

Commit message: Add mounting holes
Parts:
- added H1, H2, H3, H4: (no value), symbol Mechanical:MountingHole
Other:
- note added: "Mounting"
- note added: "USB-C Power Delivery"
- note added: "negotiates 20V Caution: There is no current capability checking."
- note removed: "USB-C Power Delivery negotiates 20V Caution: There is no current capability checking."
Changed lines of the file:
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@@
+    (stroke (width 0) (type default) (color 0 0 0 0))
+  )
+  (polyline (pts (xy 21.59 139.065) (xy 48.895 139.065))
     (stroke (width 0) (type default) (color 0 0 0 0))
   )
@@
     (stroke (width 0) (type default) (color 0 0 0 0))
   )
+  (polyline (pts (xy 21.59 139.065) (xy 21.59 149.86))
+    (stroke (width 0) (type default) (color 0 0 0 0))
+  )
   (wire (pts (xy 25.4 127) (xy 25.4 128.27))
     (stroke (width 0) (type default) (color 0 0 0 0))
@@
     (stroke (width 0) (type default) (color 0 0 0 0))
   )
+  (polyline (pts (xy 48.895 149.86) (xy 48.895 139.065))
+    (stroke (width 0) (type default) (color 0 0 0 0))
+  )
   (wire (pts (xy 175.26 102.87) (xy 175.26 107.95))
     (stroke (width 0) (type default) (color 0 0 0 0))
@@
     (stroke (width 0) (type default) (color 0 0 0 0))
   )
+  (polyline (pts (xy 21.59 149.86) (xy 48.895 149.86))
+    (stroke (width 0) (type default) (color 0 0 0 0))
+  )
   (wire (pts (xy 60.96 107.95) (xy 60.96 110.49))
     (stroke (width 0) (type default) (color 0 0 0 0))
@@
   (polyline (pts (xy 110.49 148.59) (xy 172.72 148.59))
     (stroke (width 0) (type default) (color 0 0 0 0))
+  )
+  (text "USB-C Power Delivery" (at 22.86 79.375 0)
+    (effects (font (size 1.27 1.27) (thickness 0.254) bold italic) (justify left bottom))
   )
   (text "If no voltage is given, then these caps are rated for 6.3V\n\n"
@@
     (effects (font (size 2.54 2.54)) (justify left bottom))
   )
-  (text "USB-C Power Delivery\nnegotiates 20V\nCaution: There is no current \ncapability checking.\n"
+  (text "negotiates 20V\nCaution: There is no current \ncapability checking.\n"
     (at 102.87 116.84 0)
     (effects (font (size 1.27 1.27)) (justify right bottom))
+  )
+  (text "Mounting" (at 22.86 141.605 0)
+    (effects (font (size 1.27 1.27) (thickness 0.254) bold italic) (justify left bottom))
   )
   (text "INTV_{CC} = 5.4V\nR_{blue}: R = (5.4V - 3.0V) / 12.5mA = 192 Ohm -> 180 Ohm\nR_{green}: R = (5.4V - 2.0V) / 10mA = 340 Ohm -> 330 Ohm\nR_{red}: R = (5.4V - 2.0V) / 20mA = 170 Ohm -> 180 Ohm"
@@
     (pin "2")
   )
+  (symbol (lib_id "Mechanical:MountingHole") (at 31.75 145.415 0) (unit 1)
+    (in_bom yes) (on_board yes)
+    (property "Reference" "H2" (id 0) (at 33.02 146.685 0)
+      (effects (font (size 1.27 1.27)) (justify left))
+    )
+    (property "Value" "" (id 1) (at 34.29 146.4818 0)
+      (effects (font (size 1.27 1.27)) (justify left) hide)
+    )
+    (property "Footprint" "" (id 2) (at 31.75 145.415 0)
+      (effects (font (size 1.27 1.27)) hide)
+    )
+    (property "Datasheet" "~" (id 3) (at 31.75 145.415 0)
+      (effects (font (size 1.27 1.27)) hide)
+    )
+  )
   (symbol (lib_id "Device:R") (at 146.05 118.11 0) (unit 1)
     (in_bom yes) (on_board yes) (fields_autoplaced)
@@
     (pin "2")
   )
+  (symbol (lib_id "Mechanical:MountingHole") (at 38.1 145.415 0) (unit 1)
+    (in_bom yes) (on_board yes)
+    (property "Reference" "H3" (id 0) (at 39.37 146.685 0)
+      (effects (font (size 1.27 1.27)) (justify left))
+    )
+    (property "Value" "" (id 1) (at 40.64 146.4818 0)
+      (effects (font (size 1.27 1.27)) (justify left) hide)
+    )
+    (property "Footprint" "" (id 2) (at 38.1 145.415 0)
+      (effects (font (size 1.27 1.27)) hide)
+    )
+    (property "Datasheet" "~" (id 3) (at 38.1 145.415 0)
+      (effects (font (size 1.27 1.27)) hide)
+    )
+  )
   (symbol (lib_id "Device:R") (at 135.89 118.11 0) (unit 1)
     (in_bom yes) (on_board yes) (fields_autoplaced)
@@
     (pin "1")
     (pin "2")
+  )
+  (symbol (lib_id "Mechanical:MountingHole") (at 25.4 145.415 0) (unit 1)
+    (in_bom yes) (on_board yes)
+    (property "Reference" "H1" (id 0) (at 26.67 146.685 0)
+      (effects (font (size 1.27 1.27)) (justify left))
+    )
+    (property "Value" "" (id 1) (at 27.94 146.4818 0)
+      (effects (font (size 1.27 1.27)) (justify left) hide)
+    )
+    (property "Footprint" "" (id 2) (at 25.4 145.415 0)
+      (effects (font (size 1.27 1.27)) hide)
+    )
+    (property "Datasheet" "~" (id 3) (at 25.4 145.415 0)
+      (effects (font (size 1.27 1.27)) hide)
+    )
   )
   (symbol (lib_id "extraSymbols:IP2721") (at 81.28 91.44 0) (unit 1)
@@
     (pin "2")
   )
+  (symbol (lib_id "Mechanical:MountingHole") (at 44.45 145.415 0) (unit 1)
+    (in_bom yes) (on_board yes)
+    (property "Reference" "H4" (id 0) (at 45.72 146.685 0)
+      (effects (font (size 1.27 1.27)) (justify left))
+    )
+    (property "Value" "" (id 1) (at 46.99 146.4818 0)
+      (effects (font (size 1.27 1.27)) (justify left) hide)
+    )
+    (property "Footprint" "" (id 2) (at 44.45 145.415 0)
+      (effects (font (size 1.27 1.27)) hide)
+    )
+    (property "Datasheet" "~" (id 3) (at 44.45 145.415 0)
+      (effects (font (size 1.27 1.27)) hide)
+    )
+  )
   (symbol (lib_id "Device:R") (at 60.96 102.87 0) (unit 1)
     (in_bom yes) (on_board yes)
@@
       (reference "F2") (unit 1) (value "Fuse") (footprint "extraFootprints:KEYSTONE-FUSE-3557-2")
     )
+    (path "/c50d6d45-acbd-41da-8eee-ed879a037d0f"
+      (reference "H1") (unit 1) (value "~") (footprint "extraFootprints:MountingHole_3.2mm_M3_ISO7380_Keepout")
+    )
+    (path "/1ecc4c89-2823-47c6-98e1-585933d2cc77"
+      (reference "H2") (unit 1) (value "~") (footprint "extraFootprints:MountingHole_3.2mm_M3_ISO7380_Keepout")
+    )
+    (path "/67bd47e8-af67-472b-b645-49bed30d5f1a"
+      (reference "H3") (unit 1) (value "~") (footprint "extraFootprints:MountingHole_3.2mm_M3_ISO7380_Keepout")
+    )
+    (path "/e260b958-e1c5-40d1-a2f3-6370d4a1489f"
+      (reference "H4") (unit 1) (value "~") (footprint "extraFootprints:MountingHole_3.2mm_M3_ISO7380_Keepout")
+    )
     (path "/00000000-0000-0000-0000-000061abada4"

Commit message: [WIP] Start PCB
Parts:
- H1, H2, H3, H4: value (none) -> ~; footprint (none) -> extraFootprints:MountingHole_3.2mm_M3_ISO7380_Keepout
Changed lines of the file:
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@@
 (kicad_sch (version 20211123) (generator eeschema)
   (paper "A4")
-  (junction (at 63.5 87.63) (diameter 0) (color 0 0 0 0)
-  )
   (junction (at 33.02 128.27) (diameter 0) (color 0 0 0 0)
   )
@@
     (stroke (width 0) (type default) (color 0 0 0 0))
   )
+  (wire (pts (xy 63.5 87.63) (xy 63.5 88.9))
+    (stroke (width 0) (type default) (color 0 0 0 0))
+  )
   (wire (pts (xy 201.93 124.46) (xy 201.93 125.73))
     (stroke (width 0) (type default) (color 0 0 0 0))
@@
     (stroke (width 0) (type default) (color 0 0 0 0))
   )
+  (wire (pts (xy 124.46 121.92) (xy 124.46 123.19))
+    (stroke (width 0) (type default) (color 0 0 0 0))
+  )
   (wire (pts (xy 58.42 88.9) (xy 63.5 88.9))
     (stroke (width 0) (type default) (color 0 0 0 0))
   )
-  (wire (pts (xy 124.46 121.92) (xy 124.46 123.19))
+  (wire (pts (xy 146.05 113.03) (xy 146.05 114.3))
     (stroke (width 0) (type default) (color 0 0 0 0))
   )
@@
     (stroke (width 0) (type default) (color 0 0 0 0))
   )
-  (wire (pts (xy 146.05 113.03) (xy 146.05 114.3))
-    (stroke (width 0) (type default) (color 0 0 0 0))
-  )
-  (wire (pts (xy 63.5 86.995) (xy 63.5 87.63))
-    (stroke (width 0) (type default) (color 0 0 0 0))
-  )
   (wire (pts (xy 146.05 132.08) (xy 153.67 132.08))
     (stroke (width 0) (type default) (color 0 0 0 0))
@@
   )
   (wire (pts (xy 59.69 91.44) (xy 59.69 93.98))
-    (stroke (width 0) (type default) (color 0 0 0 0))
-  )
-  (wire (pts (xy 63.5 87.63) (xy 63.5 88.9))
     (stroke (width 0) (type default) (color 0 0 0 0))
   )
@@
       (effects (font (size 1.27 1.27)) (justify left))
     )
-    (property "Value" "" (id 1) (at 34.29 146.4818 0)
+    (property "Value" "~" (id 1) (at 34.29 146.4818 0)
       (effects (font (size 1.27 1.27)) (justify left) hide)
     )
-    (property "Footprint" "" (id 2) (at 31.75 145.415 0)
+    (property "Footprint" "extraFootprints:MountingHole_3.2mm_M3_ISO7380_Keepout" (id 2) (at 31.75 145.415 0)
       (effects (font (size 1.27 1.27)) hide)
     )
@@
       (effects (font (size 1.27 1.27)) (justify left))
     )
-    (property "Value" "" (id 1) (at 40.64 146.4818 0)
+    (property "Value" "~" (id 1) (at 40.64 146.4818 0)
       (effects (font (size 1.27 1.27)) (justify left) hide)
     )
-    (property "Footprint" "" (id 2) (at 38.1 145.415 0)
+    (property "Footprint" "extraFootprints:MountingHole_3.2mm_M3_ISO7380_Keepout" (id 2) (at 38.1 145.415 0)
       (effects (font (size 1.27 1.27)) hide)
     )
@@
       (effects (font (size 1.27 1.27)) (justify left))
     )
-    (property "Value" "" (id 1) (at 27.94 146.4818 0)
+    (property "Value" "~" (id 1) (at 27.94 146.4818 0)
       (effects (font (size 1.27 1.27)) (justify left) hide)
     )
-    (property "Footprint" "" (id 2) (at 25.4 145.415 0)
+    (property "Footprint" "extraFootprints:MountingHole_3.2mm_M3_ISO7380_Keepout" (id 2) (at 25.4 145.415 0)
       (effects (font (size 1.27 1.27)) hide)
     )
@@
       (effects (font (size 1.27 1.27)) (justify left))
     )
-    (property "Value" "" (id 1) (at 46.99 146.4818 0)
+    (property "Value" "~" (id 1) (at 46.99 146.4818 0)
       (effects (font (size 1.27 1.27)) (justify left) hide)
     )
-    (property "Footprint" "" (id 2) (at 44.45 145.415 0)
-      (effects (font (size 1.27 1.27)) hide)
-    )
+    (property "Footprint" "extraFootprints:MountingHole_3.2mm_M3_ISO7380_Keepout" (id 2) (at 44.45 145.415 0)
+      (effects (font (size 1.27 1.27)) hide)
+    )

Commit message: Fix wrong battery polarity Enable voltage monitoring at 15V Add caps to OFB and BFB Use another diodes Replace 1206 shunt with 0805 Replace main mosfet with bigger one Improve traces/ground planes
Parts:
- J2: symbol Connector:Conn_01x02_Female -> Connector:Conn_01x02_Socket
Connections:
- net GND: now also J2.1 (Pin_1); no longer J2.2 (Pin_2)
- net at F2.2: now also J2.2 (Pin_2); no longer J2.1 (Pin_1)
Other:
- sheet Boost-Converter ports: added RUN; removed SS
Changed lines of the file:
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@@
     )
   )
-  (symbol (lib_id "Connector:Conn_01x02_Female") (at 208.28 121.92 0) (unit 1)
-    (in_bom yes) (on_board yes) (dnp no) (fields_autoplaced)
-    (property "Reference" "J2" (at 208.9912 122.3553 0)
-      (effects (font (size 1.27 1.27)) (justify left))
-    )
-    (property "Value" "BatteryConnection" (at 208.9912 124.8922 0)
-      (effects (font (size 1.27 1.27)) (justify left))
-    )
-    (property "Footprint" "Connector_AMASS:AMASS_XT30U-M_1x02_P5.0mm_Vertical" (at 208.28 121.92 0)
-      (effects (font (size 1.27 1.27)) hide)
-    )
-    (property "Datasheet" "~" (at 208.28 121.92 0)
+  (symbol (lib_id "Connector:Conn_01x02_Socket") (at 208.28 124.46 0) (mirror x) (unit 1)
+    (in_bom yes) (on_board yes) (dnp no)
+    (property "Reference" "J2" (at 208.9912 124.0247 0)
+      (effects (font (size 1.27 1.27)) (justify left))
+    )
+    (property "Value" "BatteryConnection" (at 208.9912 121.4878 0)
+      (effects (font (size 1.27 1.27)) (justify left))
+    )
+    (property "Footprint" "Connector_AMASS:AMASS_XT30U-M_1x02_P5.0mm_Vertical" (at 208.28 124.46 0)
+      (effects (font (size 1.27 1.27)) hide)
+    )
+    (property "Datasheet" "~" (at 208.28 124.46 0)
       (effects (font (size 1.27 1.27)) hide)
     )
@@
       (effects (font (size 1.27 1.27)) (justify left))
     )
-    (pin "SS" input (at 171.45 102.87 270)
-      (effects (font (size 1.27 1.27)) (justify left))
-    )
     (pin "INTV_{CC}" output (at 168.91 96.52 180)
       (effects (font (size 1.27 1.27)) (justify left))
     )
+    (pin "RUN" input (at 171.45 102.87 270)
+      (effects (font (size 1.27 1.27)) (justify left))
+    )
